File: PCB/MasterModule/MasterModule.kicad_sch (KiCad schematic)
At the start: 10 parts, among them Con1 Male Connector, Con2 Femail Connector, P1 USB Power

Commit message: PCB update
Parts:
- added U1: I2C Level Shifter, 7_Segment_Clock_Footprint_Library:I2C_Level_Shifter, symbol 7_Segment_Clock_Symbol_Library:I2C_Level_Shifter
- added U2: ESP32, 7_Segment_Clock_Footprint_Library:ESP32_Connection_Footprint, symbol 7_Segment_Clock_Symbol_Library:ESP32_Connection
- Con1, Con2: footprint (none) -> 7_Segment_Clock_Footprint_Library:JST_Connector_Footprint
- P1: footprint (none) -> 7_Segment_Clock_Footprint_Library:Power_Connection_Footprint
Connections:
- net +5V: now also R3.1, U1.1 (VCC), U2.1 (5V)
- net GND: now also U1.4 (GND), U1.8 (GND), U2.2 (GND)
- net SCL 5V: now also U1.3 (SCL)
- net SDA 5V: now also U1.2 (SDA)
- new net +3V3: U1.5 (VCC), U2.3 (3V3)
- new net SCL 3V3: U1.7 (SCL), U2.5 (SCL)
- new net SDA 3V3: U1.6 (SDA), U2.4 (SDA)

Commit message: PCB update
Parts:
- added C1: 1000uf, Capacitor_THT:C_Radial_D6.3mm_H7.0mm_P2.50mm, symbol Device:C_Polarized
- added C2, C3: 100nf, Capacitor_THT:C_Disc_D3.0mm_W2.0mm_P2.50mm, symbol Device:C
- added U3: ESP32 Signals, Connector_PinHeader_2.54mm:PinHeader_1x05_P2.54mm_Vertical, symbol 7_Segment_Clock_Symbol_Library:ESP32_Signal_Connection
- added U4: Controls, Connector_PinHeader_2.54mm:PinHeader_1x06_P2.54mm_Vertical, symbol 7_Segment_Clock_Symbol_Library:Control_Connections
- L1, L2, L3: footprint 7_Segment_Clock_Footprint_Library:LED_Connection_Footprint -> Connector_PinHeader_2.54mm:PinHeader_1x02_P2.54mm_Vertical
- U2: footprint 7_Segment_Clock_Footprint_Library:ESP32_Connection_Footprint -> Connector_PinHeader_2.54mm:PinHeader_1x05_P2.54mm_Vertical
Connections:
- net +5V: now also C1.1, C2.2, C3.1
- net GND: now also C1.2, C2.1, C3.2, U4.4 (GND), U4.5 (GND), U4.6 (GND)
- net at R2.2: now also U3.5 (LED2)
- net at R1.2: now also U3.4 (LED1)
- new net: U3.1 (Btn1), U4.1 (Btn1)
- new net: U3.2 (Btn2), U4.2 (Btn2)
- new net: U3.3 (SW), U4.3 (Sw)
Other:
- moved on the sheet: U2

Commit message: Created (and ordered) the pcb
Parts:
- added R4, R5, R6, R7: 4k7, Resistor_THT:R_Axial_DIN0204_L3.6mm_D1.6mm_P7.62mm_Horizontal, symbol Device:R
- C1: footprint Capacitor_THT:C_Radial_D6.3mm_H7.0mm_P2.50mm -> Capacitor_THT:C_Radial_D8.0mm_H11.5mm_P3.50mm
- R1, R2, R3: footprint Resistor_THT:R_Axial_DIN0204_L3.6mm_D1.6mm_P5.08mm_Horizontal -> Resistor_THT:R_Axial_DIN0204_L3.6mm_D1.6mm_P7.62mm_Horizontal
Connections:
- net +3V3: now also R4.1, R5.2
- net +5V: now also C2.1, RTC1.2 (VCC), R6.2, R7.2; no longer C2.2, RTC1.1 (VCC)
- net GND: now also C2.2, RTC1.1 (GND), U1.2 (GND), U1.6 (GND); no longer C2.1, RTC1.2 (GND), U1.4 (GND), U1.8 (GND)
- net SCL 3V3: now also U1.8 (SCL), R5.1; no longer U1.7 (SCL)
- net SCL 5V: now also U1.4 (SCL), R6.1; no longer U1.3 (SCL)
- net SDA 3V3: now also U1.7 (SDA), R4.2; no longer U1.6 (SDA)
- net SDA 5V: now also U1.3 (SDA), R7.1; no longer U1.2 (SDA)
Other:
- moved on the sheet: C2
